Commit message: [xslocobot_descriptions] Replace Realsense with ZED

File: interbotix_ros_xslocobots/interbotix_xslocobot_descriptions/urdf/locobot.urdf.xacro (robot description, xacro)
@@ -18,4 +18,14 @@
   <xacro:property name="urdf_loc"         value="$(arg external_urdf_loc)"/>
   <xacro:property name="pi_offset"        value="0.00001"/>
+  <!-- ZED camera -->
+  <xacro:arg name="camera_name"   default="zed2" />
+  <xacro:arg name="camera_model"  default="zed2" />
+  <xacro:arg name="base_frame"    default="locobot/tilt_link" />
+  <xacro:arg name="cam_pos_x"     default="0.05318" />
+  <xacro:arg name="cam_pos_y"     default="0.0175" />
+  <xacro:arg name="cam_pos_z"     default="0.000009" />
+  <xacro:arg name="cam_roll"      default="0.0" />
+  <xacro:arg name="cam_pitch"     default="0.0" />
+  <xacro:arg name="cam_yaw"       default="0.0" />
   <xacro:if value="${urdf_loc != ''}">
     <xacro:include filename="${urdf_loc}"/>

File: interbotix_ros_xslocobots/interbotix_xslocobot_descriptions/urdf/pan_and_tilt.urdf.xacro (robot description, xacro)
@@ -137,5 +137,5 @@
       <self_collide>true</self_collide>
     </gazebo>
-    <joint name="camera" type="fixed">
+    <!-- <joint name="camera" type="fixed">
       <origin
         rpy="0 0 0"
@@ -144,10 +144,17 @@
         link="${robot_name}/tilt_link"/>
       <child
-        link="camera_${robot_name}_link"/>
-    </joint>
+        link="$(arg camera_name)_base_link"/>
+    </joint> -->
+    <!-- <link name="${arg camera_name}_base_link" /> -->
+    <xacro:include filename="$(find interbotix_xslocobot_descriptions)/urdf/zed_camera/zed_macro.urdf.xacro" />
+    <xacro:zed_camera name="$(arg camera_name)" model="$(arg camera_model)" parent="$(arg base_frame)">
+        <origin
+          xyz="$(arg cam_pos_x) $(arg cam_pos_y) $(arg cam_pos_z)"
+          rpy="$(arg cam_roll) $(arg cam_pitch) $(arg cam_yaw)"/>
+    </xacro:zed_camera>
     <gazebo reference="camera">
       <disableFixedJointLumping>true</disableFixedJointLumping>
     </gazebo>
-    <link name="camera_${robot_name}_link">
+    <!-- <link name="camera_${robot_name}_link">
       <visual>
         <origin
@@ -187,5 +194,5 @@
           izz="0.0000468600"/>
       </inertial>
-    </link>
+    </link> -->
     <gazebo reference="camera_${robot_name}_link">
       <material>Gazebo/Grey</material>
@@ -194,5 +201,5 @@
     <!-- Adds a dummy link, libgazebo_ros_openni_kinect publishes from frame's z-axis -->
     <!-- https://github.com/ros-simulation/gazebo_ros_pkgs/issues/243 -->
-    <joint name="camera_depth_joint" type="fixed">
+    <!-- <joint name="camera_depth_joint" type="fixed">
       <origin rpy="${-pi/2} 0 ${-pi/2}" xyz="0 0 0"/>
       <parent link="camera_${robot_name}_link"/>
@@ -201,5 +208,5 @@
     <link name="${robot_name}/camera_depth_link">
       <origin rpy="0 0 0" xyz="0 0 0"/>
-    </link>
+    </link> -->
     <gazebo reference="camera_${robot_name}_link">
       <sensor name="camera_frame_sensor" type="depth">
